File: matrix.kicad_sch (KiCad schematic)
At the start: 98 parts, among them SW1 choc_v1_SW_HS, SW10 choc_v1_SW_HS, SW11 choc_v1_SW_HS, SW12 choc_v1_SW_HS, SW13 choc_v1_SW_HS, SW14 choc_v1_SW_HS, SW15 choc_v1_SW_HS, SW16 choc_v1_SW_HS, SW17 choc_v1_SW_HS, SW18 choc_v1_SW_HS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

Commit message: drc errors fix
Parts:
- SW42: footprint Library:SW_choc_v2_HS_CPG135001S30_1u_switch_hide -> Library:SW_choc_v2_HS_CPG135001S30_1u_SW42
- SW43: footprint Library:SW_choc_v2_HS_CPG135001S30_1u -> Library:SW_choc_v2_HS_CPG135001S30_1u_SW42_switch_show
