File: koiboard2.kicad_pcb (KiCad board)
At the start: 4 copper layers, 227 x 75.4 mm, 138 parts, among them J1 USB_C_Receptacle_USB2.0_16P, SW1 choc_v1_SW_HS, SW10 choc_v1_SW_HS, SW11 choc_v1_SW_HS, SW12 choc_v1_SW_HS, SW13 choc_v1_SW_HS, SW14 choc_v1_SW_HS, SW15 choc_v1_SW_HS, SW16 choc_v1_SW_HS, SW17 choc_v1_SW_HS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

Commit message: BOM
Routing:
- net GND: vias 48 -> 49
