File: pcb/koiboard2_4layer.kicad_pcb (KiCad board)
At the start: 2 copper layers, 227 x 75.4 mm, 138 parts, among them J1 USB_C_Receptacle_USB2.0_16P, SW1 choc_v1_SW_HS, SW10 choc_v1_SW_HS, SW11 choc_v1_SW_HS, SW12 choc_v1_SW_HS, SW13 choc_v1_SW_HS, SW14 choc_v1_SW_HS, SW15 choc_v1_SW_HS, SW16 choc_v1_SW_HS, SW17 choc_v1_SW_HS, SW18 choc_v1_SW_HS, SW19 choc_v1_SW_HS, SW2 choc_v1_SW_HS, SW20 choc_v1_SW_HS, SW21 choc_v1_SW_HS, SW22 choc_v1_SW_HS, SW23 choc_v1_SW_HS, SW24 choc_v1_SW_HS, SW25 choc_v1_SW_HS, SW26 choc_v1_SW_HS, SW27 choc_v1_SW_HS, SW28 choc_v1_SW_HS, SW29 choc_v1_SW_HS, SW3 choc_v1_SW_HS, SW30 choc_v1_SW_HS, SW31 choc_v1_SW_HS, SW32 choc_v1_SW_HS, SW33 choc_v1_SW_HS, SW34 choc_v1_SW_HS, SW35 choc_v1_SW_HS, SW36 choc_v1_SW_HS, SW37 choc_v1_SW_HS, SW38 choc_v1_SW_HS, SW39 choc_v1_SW_HS, SW4 choc_v1_SW_HS, SW40 choc_v1_SW_HS, SW41 choc_v1_SW_HS, SW42 choc_v1_SW_HS, SW43 choc_v1_SW_HS, SW44 choc_v1_SW_HS, SW45 choc_v1_SW_HS, SW46 choc_v1_SW_HS, SW47 choc_v1_SW_HS, SW48 choc_v1_SW_HS, SW49 choc_v1_SW_HS, SW5 choc_v1_SW_HS, SW6 choc_v1_SW_HS, SW7 choc_v1_SW_HS, SW8 choc_v1_SW_HS, SW9 choc_v1_SW_HS, U1 XC6206PxxxMR, U2 SRV05-4, U3 RP2040, U4 W25Q128JVS, Y1 Crystal_GND24

Commit message: 2 layer final
Parts:
- moved C4 1.91 mm to (131.8, 53.6), turned to 135 degrees
- moved F1 0.96 mm to (131.0, 31.7)
Connections:
- net D2+ renamed Net-(U3-USB_DP)
- net D2- renamed Net-(U3-USB_DM)
Routing:
- net +3V3: track 188.2 -> 41.8 mm, vias 10 -> 8
- net +1V1: track 26.9 -> 20.1 mm
- net COL5: track 88.8 -> 82.1 mm
- net +5V: track 13.3 -> 9.48 mm, vias 2 -> 0
- net COL6: track 65.7 -> 69.4 mm
- net D+: track 31.1 -> 28.6 mm
- net GND: track 7.29 -> 5.44 mm, vias 63 -> 49
- net COL0: track 159.8 -> 158.3 mm
- net COL8: track 102.3 -> 101.0 mm
- net D-: track 30.0 -> 28.8 mm
- net COL7: track 87.6 -> 86.5 mm
- net COL1: track 150.3 -> 149.2 mm
- net COL3: track 116.1 -> 115.1 mm
- net COL10: track 140.6 -> 139.6 mm
- net COL4: track 103.0 -> 102.2 mm
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- added copper zone on In1.Cu, net +1V1
- added copper zone on In1.Cu, net +3V3
- added copper zone on In2.Cu, net GND
Other:
- copper layers 2 -> 4
